File: pcb_piano/pcb_piano_v1.kicad_pcb (KiCad board)
At the start: 2 copper layers, 60 parts, among them P1 CONN_01X06_M50-3530642, P2 CONN_01X06_M50-3530642, U1 connex_EFM32HG322F64G-B-QFP48, U2 connex-accel-LIS2DHTR, U3 CONNEX_REGUL_LT4081, U4 CONNEX-DIODE-TVS-USB-USBLC6-4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, Y1 Crystal_8MHZ_ABM3B-8.000MHZ-B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

Commit message: Pushed Version 1 hardware
Parts:
- removed P2: CONN_01X06_M50-3530642, Pin_Headers:Pin_Header_Straight_1x06
- added D1: LED_RGB_SMLP34RGB1W3, connex_led:led_0404_SMLP34RGB1W3, F.Cu at (102.4, 52.3)
- added D2: LED_RGB_SMLP34RGB1W3, connex_led:led_0404_SMLP34RGB1W3, F.Cu at (95.0, 51.8)
- added FB2: CONNEX-SMD-FERRITE-BEAD-300MA-BLM15AG102SN1D, connex_inductor:L_0402, F.Cu at (64.2, 56.8)
- added G***: LOGO, connex_logo:chicken_outline_12mmx15mm, F.Cu at (142.0, 92.0)
- added G***: LOGO, connex_logo:chicken_outline_12mmx15mm, F.Cu at (121.0, 92.0)
- added G***: LOGO, connex_logo:chicken_outline_12mmx15mm, F.Cu at (100.0, 92.0)
- added G***: LOGO, connex_logo:chicken_outline_12mmx15mm, F.Cu at (79.0, 92.0)
- added G***: LOGO, connex_logo:chicken_outline_12mmx15mm, F.Cu at (58.6, 91.8)
- added J1: CONNEX_CONN_2PIN_KEYED, connex_connectors:CONNEX_CONN-2POS-KEYED-S2B-PH-K-S, F.Cu at (79.7, 54.9)
- added Q1: Q_NMOS_SSM3K09FULF, TO_SOT_Packages_SMD:SC-70, F.Cu at (72.0, 56.7)
- added R24: CONNEX-SMD-RES-10K-0603, Resistors_SMD:R_0603, F.Cu at (71.0, 54.5)
- added R25: CONNEX-SMD-RES-120-0603, Resistors_SMD:R_0603, F.Cu at (104.2, 55.8)
- added R26: SMD-RES-10K-1%-1_10W_0603_, Resistors_SMD:R_0603, F.Cu at (100.8, 61.1)
- added R27: CONNEX-SMD-RES-30-0603, Resistors_SMD:R_0603, F.Cu at (102.5, 55.8)
- added R28: CONNEX-SMD-RES-20-0603, Resistors_SMD:R_0603, F.Cu at (100.8, 55.8)
- added R29: CONNEX-SMD-RES-120-0603, Resistors_SMD:R_0603, F.Cu at (96.5, 55.5)
- added R30: CONNEX-SMD-RES-30-0603, Resistors_SMD:R_0603, F.Cu at (94.8, 55.5)
- added R31: CONNEX-SMD-RES-20-0603, Resistors_SMD:R_0603, F.Cu at (93.0, 55.5)
- added R32: CONNEX-SMD-RES-324K-0402, Resistors_SMD:R_0402, F.Cu at (88.0, 68.2)
- added R33: CONNEX-SMD-RES-634k-0402, Resistors_SMD:R_0402, F.Cu at (87.9, 59.9)
- added R34: CONNEX-SMD-RES-10K-0603, Resistors_SMD:R_0603, F.Cu at (67.8, 56.3)
- added R35: CONNEX-SMD-RES-10K-0603, Resistors_SMD:R_0603, F.Cu at (67.8, 58.0)
- added SP1: connex-piezo-4khz-AT-2440-TWT-R, connex_device:CONNEX-PIEZO-AT-2440-TWT-R, F.Cu at (63.8, 70.8)
- added TP10: test_point_smt, connex_diodes:TEST_POINT_SMD_50MIL, F.Cu at (100.0, 67.0)
- added TP11: test_point_smt, connex_diodes:TEST_POINT_SMD_50MIL, F.Cu at (72.0, 52.0)
- added TP4: test_point_smt, connex_diodes:TEST_POINT_SMD_50MIL, F.Cu at (113.8, 57.3)
- added TP5: test_point_smt, connex_diodes:TEST_POINT_SMD_50MIL, F.Cu at (89.4, 58.1)
- added TP6: test_point_smt, connex_diodes:TEST_POINT_SMD_50MIL, F.Cu at (77.0, 66.0)
- added TP7: test_point_smt, connex_diodes:TEST_POINT_SMD_50MIL, F.Cu at (94.2, 80.7)
- added TP8: test_point_smt, connex_diodes:TEST_POINT_SMD_50MIL, F.Cu at (100.0, 65.0)
- added TP9: test_point_smt, connex_diodes:TEST_POINT_SMD_50MIL, F.Cu at (100.0, 63.0)
- CT1, CT2, CT3, CT4, CT5: footprint connex_cap_touch:CONNEX-CAPTOUCH-SINGLE-BUTTON-20MM -> connex_cap_touch:CONNEX-CAPTOUCH-SINGLE-BUTTON-15MM
- R11: value SMD-RES-10K-1%-1_10W_0603_ -> CONNEX-SMD-RES-0-0603
- R12: value SMD-RES-0R-1_4W_0603_ -> CONNEX-SMD-RES-1M-0603
- R22: value CONNEX-SMD-RES-324K-0603 -> CONNEX-SMD-RES-324K-0402; footprint Resistors_SMD:R_0603 -> Resistors_SMD:R_0402
- TP1, TP2, TP3: footprint connex_test:TEST_POINT_SMD_50MIL -> connex_diodes:TEST_POINT_SMD_50MIL
- U2: footprint connex_smd_misc:CONNEX_DFN_10PIN_3MMX3MM -> connex_smd_misc:CONNEX_LGA-14_2MMX2MM
- moved U3 145.1 mm to (84.0, 67.2)
- moved R13 141.3 mm to (80.1, 65.2), turned to 270 degrees
- moved R12 133.5 mm to (67.8, 54.5), turned to 180 degrees
- moved R14 112.1 mm to (92.5, 63.3)
- moved R15 109.5 mm to (88.0, 65.6), turned to 90 degrees
- moved P1 104.8 mm to (120.8, 54.1), turned to 90 degrees
- moved R3 103.4 mm to (95.0, 78.5), turned to 180 degrees
- moved R19 101.2 mm to (131.0, 61.0), turned to 180 degrees
- moved TP2 99.1 mm to (91.2, 56.4), turned to 90 degrees
- moved R22 97.2 mm to (87.9, 57.7), turned to 90 degrees
- moved R18 96.9 mm to (89.8, 68.5), turned to 270 degrees
- moved R11 95.2 mm to (64.2, 54.5)
- moved C10 94.9 mm to (124.5, 64.2)
- moved R1 94.7 mm to (95.0, 72.5), turned to 180 degrees
- moved C4 92.0 mm to (120.5, 71.0), turned to 270 degrees
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Connections:
- net Net-(C12-Pad1) renamed /PWR_VDD_DREG
- net Net-(C3-Pad1) renamed /PWR_AVDD
- net Net-(C6-Pad1) renamed /PWR_IOVDD
- net Net-(FB1-Pad1) renamed /USB_VBUS_CONN
- C10 pad 1: /USB_VREG_IN -> /USB_VBUS_IN
- C17 pad 1: /3V3_CHARGE_INPUT -> /USB_VREG_IN
- P1 pad 2: /BOOT_RX -> GND
- P1 pad 3: /BOOT_TX -> /BOOT_RX
- P1 pad 4: /RESETn -> /BOOT_TX
- P1 pad 5: Net-(P1-Pad5) -> /RESETn
- P1 pad 6: /POWER_INPUT_CONN -> +3V3
- R11 pad 1: Net-(R11-Pad1) -> +3V3
- R11 pad 2: /3V3_CHARGE_INPUT -> Net-(FB2-Pad1)
- R12 pad 1: +3V3 -> Net-(Q1-Pad1)
- R12 pad 2: /USB_VREG_IN -> GND
- R13 pad 1: /USB_VREG_IN -> /USB_VBUS_IN
- R13 pad 2: /3V3_CHARGE_INPUT -> /USB_VREG_IN
- R16 pad 2: /3V3_CHARGE_INPUT -> /BATT_CONN_OUTPUT
- R19 pad 2: /USB_VREG_IN -> /USB_VBUS_IN
- R22 pad 1: Net-(R15-Pad1) -> /BATT_ADC
- R22 pad 2: GND -> /BATT_CONN_OUTPUT
- TP1 pad 1: /3V3_CHARGE_INPUT -> /UART_TX
- TP2 pad 1: Net-(R11-Pad1) -> Net-(R29-Pad2)
- U1 pad 1: Net-(U1-Pad1) -> /EN_BUCK_MCU
- U1 pad 2: Net-(U1-Pad2) -> /MODE
- U1 pad 3: Net-(U1-Pad3) -> /EN_CHRG
- U1 pad 33: /USB_VREG_IN -> /USB_VBUS_IN
- U1 pad 39: Net-(U1-Pad39) -> /STAT_LED_R
- U1 pad 40: Net-(U1-Pad40) -> /STAT_LED_B
- U1 pad 48: Net-(U1-Pad48) -> /PIEZO_PWM_MCU
- U3 pad 2: /3V3_CHARGE_INPUT -> /USB_VREG_IN
- U3 pad 6: Net-(R11-Pad1) -> Net-(R29-Pad2)
Routing:
- net GND: track 0.00 -> 421.0 mm, vias 0 -> 36
- net +3V3: track 0.00 -> 178.5 mm, vias 0 -> 2
- net /USB_VBUS_IN: track 0.00 -> 101.9 mm, vias 0 -> 2
- net /PWR_IOVDD: track 0.00 -> 80.2 mm, vias 0 -> 5
- net /CAP_TOUCH1: track 0.00 -> 68.6 mm
- net /CAP_TOUCH5: track 0.00 -> 51.3 mm
- net /PIEZO_PWM_MCU: track 0.00 -> 50.1 mm, vias 0 -> 2
- net /CAP_TOUCH2: track 0.00 -> 48.6 mm
- net /PWR_VDD_DREG: track 0.00 -> 42.8 mm, vias 0 -> 2
- net /USB_VREG_IN: track 0.00 -> 41.6 mm
- net /EN_CHRG: track 0.00 -> 39.4 mm, vias 0 -> 2
- net /BATT_ADC: track 0.00 -> 36.5 mm, vias 0 -> 2
- net /CAP_TOUCH4: track 0.00 -> 33.9 mm
- net /MODE: track 0.00 -> 33.7 mm, vias 0 -> 2
- net /PWR_AVDD: track 0.00 -> 33.5 mm, vias 0 -> 3
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- added copper zone on B.Cu, net GND
- added copper zone on F.Cu, net GND
Other:
- board outline added: 100 x 50 mm
- net class Default: clearance 0.2 -> 0.152; trace_width 0.25 -> 0.2; via_drill 0.4 -> 0.3
- rule trace_clearance: 0.2 -> 0.152
- rule trace_min: 0.2 -> 0.152
- rule via_min_size: 0.4 -> 0.6
- board text added: "CONNEX PCB PECKER PIANO REVA01 12-13-2017"
